File: KiCad/Crepuscolare.sch (KiCad schematic (older format))
At the start: 13 parts, among them K1 RELAY_1RT, Q1 BC337, U1 ARDUINO_NANO_IC

Commit message: Allineamento progetto
Parts:
- added LDR1: 5K-500K, ~, symbol LDR
- added R1: 2K7, ~, symbol RESISTOR
- added R6: 10K, ~, symbol RESISTOR
- K1: value RELAY_1RT -> HR703V
- renumbered LDR1 to LDR2, R1 to R2, R2 to R3, R3 to R4, R4 to R5
Connections:
- wire segments 32 -> 37
- no-connect marks 27 -> 26
Changed lines of the file:
@@
 Sheet 1 1
 Title "Crepuscolare con Arduino"
-Date "6 feb 2015"
+Date "8 feb 2015"
 Rev "2015-01"
 Comp ""
@@
 $EndComp
 $Comp
-L RESISTOR R2
+L RESISTOR R3
 U 1 1 54CF30A1
 P 1900 4000
-F 0 "R2" H 2050 4050 60  0000 C CNN
+F 0 "R3" H 2050 4050 60  0000 C CNN
 F 1 "47K" H 2050 3850 60  0000 C CNN
 F 2 "~" H 1900 4000 60  0000 C CNN
@@
 $EndComp
 $Comp
-L LDR LDR1
+L LDR LDR2
 U 1 1 54D465C4
 P 1900 4650
-F 0 "LDR1" H 2100 4750 60  0000 C CNN
-F 1 "5K-500K" H 2150 4400 60  0000 C CNN
+F 0 "LDR2" H 2150 4650 60  0000 C CNN
+F 1 "5K-500K" H 2150 4500 60  0000 C CNN
 F 2 "~" H 1900 4650 60  0000 C CNN
 F 3 "~" H 1900 4650 60  0000 C CNN
@@
 $EndComp
 Wire Wire Line
-	1900 3500 3200 3500
+	1300 3500 3200 3500
 Wire Wire Line
 	1900 3500 1900 3850
 $Comp
-L GND #PWR01
+L GND #PWR5
 U 1 1 54D465F2
 P 1900 5300
-F 0 "#PWR01" H 1900 5300 30  0001 C CNN
+F 0 "#PWR5" H 1900 5300 30  0001 C CNN
 F 1 "GND" H 1900 5230 30  0001 C CNN
 F 2 "" H 1900 5300 60  0000 C CNN
@@
 Connection ~ 2550 3500
 $Comp
-L GND #PWR02
+L GND #PWR6
 U 1 1 54D4661A
 P 2550 5300
-F 0 "#PWR02" H 2550 5300 30  0001 C CNN
+F 0 "#PWR6" H 2550 5300 30  0001 C CNN
 F 1 "GND" H 2550 5230 30  0001 C CNN
 F 2 "" H 2550 5300 60  0000 C CNN
@@
 P 6350 4000
 F 0 "K1" H 6450 4250 40  0000 C CNN
-F 1 "RELAY_1RT" H 6550 3900 40  0000 C CNN
+F 1 "HR703V" H 6350 4350 40  0000 C CNN
 F 2 "~" H 6350 4020 60  0000 C CNN
 F 3 "~" H 6350 4020 60  0000 C CNN
@@
 $EndComp
 $Comp
-L RESISTOR R4
+L RESISTOR R5
 U 1 1 54D46805
 P 4900 4400
-F 0 "R4" H 5050 4450 60  0000 C CNN
+F 0 "R5" H 5050 4450 60  0000 C CNN
 F 1 "510K" H 5050 4250 60  0000 C CNN
 F 2 "~" H 4900 4400 60  0000 C CNN
@@
 $EndComp
 $Comp
-L RESISTOR R1
+L RESISTOR R2
 U 1 1 54D4680B
 P 5850 3750
-F 0 "R1" H 5700 3800 60  0000 C CNN
+F 0 "R2" H 5700 3800 60  0000 C CNN
 F 1 "470" H 5700 3650 60  0000 C CNN
 F 2 "~" H 5850 3750 60  0000 C CNN
@@
 $EndComp
 $Comp
-L GND #PWR03
+L GND #PWR7
 U 1 1 54D46825
 P 4900 5300
-F 0 "#PWR03" H 4900 5300 30  0001 C CNN
+F 0 "#PWR7" H 4900 5300 30  0001 C CNN
 F 1 "GND" H 4900 5230 30  0001 C CNN
 F 2 "" H 4900 5300 60  0000 C CNN
@@
 $EndComp
 $Comp
-L GND #PWR04
+L GND #PWR8
 U 1 1 54D4682B
 P 5850 5300
-F 0 "#PWR04" H 5850 5300 30  0001 C CNN
+F 0 "#PWR8" H 5850 5300 30  0001 C CNN
 F 1 "GND" H 5850 5230 30  0001 C CNN
 F 2 "" H 5850 5300 60  0000 C CNN
@@
 	5300 4800 5550 4800
 $Comp
-L RESISTOR R3
+L RESISTOR R4
 U 1 1 54D46887
 P 5300 4350
-F 0 "R3" H 5450 4400 60  0000 C CNN
+F 0 "R4" H 5450 4400 60  0000 C CNN
 F 1 "2K7" H 5450 4200 60  0000 C CNN
 F 2 "~" H 5300 4350 60  0000 C CNN
@@
 $EndComp
 $Comp
-L GND #PWR05
+L GND #PWR2
 U 1 1 54D469B8
 P 2650 2800
-F 0 "#PWR05" H 2650 2800 30  0001 C CNN
+F 0 "#PWR2" H 2650 2800 30  0001 C CNN
 F 1 "GND" H 2650 2730 30  0001 C CNN
 F 2 "" H 2650 2800 60  0000 C CNN
@@
 NoConn ~ 3200 4550
 NoConn ~ 3200 4400
-NoConn ~ 3200 4250
 NoConn ~ 3200 4100
 NoConn ~ 3200 3950
@@
 	4700 3500 4450 3500
 $Comp
-L GND #PWR06
+L GND #PWR3
 U 1 1 54D46C10
 P 4700 3600
-F 0 "#PWR06" H 4700 3600 30  0001 C CNN
+F 0 "#PWR3" H 4700 3600 30  0001 C CNN
 F 1 "GND" H 4700 3530 30  0001 C CNN
 F 2 "" H 4700 3600 60  0000 C CNN
@@
 $EndComp
 $Comp
-L +9V #PWR07
+L +9V #PWR1
 U 1 1 54D46CEA
 P 3050 2150
-F 0 "#PWR07" H 3050 2120 20  0001 C CNN
+F 0 "#PWR1" H 3050 2120 20  0001 C CNN
 F 1 "+9V" H 3050 2260 30  0000 C CNN
 F 2 "" H 3050 2150 60  0000 C CNN
@@
 $EndComp
 $Comp
-L PWR_FLAG #FLG08
+L PWR_FLAG #FLG2
 U 1 1 54D46D52
 P 3300 2200
-F 0 "#FLG08" H 3300 2295 30  0001 C CNN
+F 0 "#FLG2" H 3300 2295 30  0001 C CNN
 F 1 "PWR_FLAG" H 3300 2380 30  0000 C CNN
 F 2 "" H 3300 2200 60  0000 C CNN
@@
 	3050 3050 3200 3050
 $Comp
-L PWR_FLAG #FLG09
+L PWR_FLAG #FLG1
 U 1 1 54D47080
 P 2650 2200
-F 0 "#FLG09" H 2650 2295 30  0001 C CNN
+F 0 "#FLG1" H 2650 2295 30  0001 C CNN
 F 1 "PWR_FLAG" H 2650 2380 30  0000 C CNN
 F 2 "" H 2650 2200 60  0000 C CNN
@@
 	3300 2300 3050 2300
 Connection ~ 3050 2300
+$Comp
+L RESISTOR R6
+U 1 1 54D78395
+P 1300 4950
+F 0 "R6" H 1450 5000 60  0000 C CNN
+F 1 "10K" H 1450 4900 60  0000 C CNN
+F 2 "~" H 1300 4950 60  0000 C CNN
+F 3 "~" H 1300 4950 60  0000 C CNN
+	1    1300 4950
+	1    0    0    -1
+$EndComp
+$Comp
+L LDR LDR1
+U 1 1 54D7839B
+P 1300 4050
+F 0 "LDR1" H 1550 4100 60  0000 C CNN
+F 1 "5K-500K" H 1600 3950 60  0000 C CNN
+F 2 "~" H 1300 4050 60  0000 C CNN
+F 3 "~" H 1300 4050 60  0000 C CNN
+	1    1300 4050
+	1    0    0    -1
+$EndComp
+$Comp
+L RESISTOR R1
+U 1 1 54D783B5
+P 1300 3700
+F 0 "R1" H 1450 3750 60  0000 C CNN
+F 1 "2K7" H 1450 3600 60  0000 C CNN
+F 2 "~" H 1300 3700 60  0000 C CNN
+F 3 "~" H 1300 3700 60  0000 C CNN
+	1    1300 3700
+	1    0    0    -1
+$EndComp
+Wire Wire Line
+	1300 4250 3200 4250
+Connection ~ 1900 4250
+Wire Wire Line
+	1300 3500 1300 3550
+Connection ~ 1900 3500
+Wire Wire Line
+	1300 3850 1300 3900
+Wire Wire Line
+	1300 4200 1300 4800
+$Comp
+L GND #PWR4
+U 1 1 54D784A2
+P 1300 5300
+F 0 "#PWR4" H 1300 5300 30  0001 C CNN
+F 1 "GND" H 1300 5230 30  0001 C CNN
+F 2 "" H 1300 5300 60  0000 C CNN
+F 3 "" H 1300 5300 60  0000 C CNN
+	1    1300 5300
+	1    0    0    -1
+$EndComp
+Wire Wire Line
+	1300 5100 1300 5300
+Connection ~ 1300 4250
 $EndSCHEMATC
